File: pcb/aquarius-plus.kicad_pcb (KiCad board)
At the start: 2 copper layers, 160 x 115 mm, 217 parts, among them J1 Cassette in, J10 Audio out, J11 Hand controller 2, J12 ESP USB Host, J13 Power in, J14 FPGA spare, J15 Expansion port, J16 ESP32 spare, J2 Cassette out, J3 SD_Card, J4 Printer, J5 Hand controller 1, J6 VGA, J7 DBG, J8 USB_A, J9 USB_A, Q1 BC847C, Q2 BC847C, SW1 SW_DPDT_x2, U1 XC3S200-4TQG144, U10 IS61C5128AS-25QLI, U11 74LVC4245APW, U12 74HC166, U13 SST39SF020A-55-4C-WHE, U14 74LVC4245APW, U15 LDL1117S33R, U16 MCP1700T-2502E/TT, U17 LD1117S12, U2 SN74CBTD3861PWR, U3 MAX3221ECPWR, U4 SN74CBTD3861PWR, U5 ESP32-S2-SOLO-N4R2, U6 SN74CBTD3861PWR, U7 Z84C0010AEG, U8 SN74CBTD3861PWR, U9 74HC166, X1 SG-5032CAN, X2 SG-5032CAN

Commit message: Working on layout.
Parts:
- moved #G1 70.7 mm to (131.0, 121.5)
- moved C54 69.9 mm to (98.0, 54.0), turned to -90 degrees
- moved J12 61.0 mm to (95.0, 45.9)
- moved J6 40.0 mm to (140.0, 35.0)
- moved R33 40.0 mm to (130.2, 55.0)
- moved R34 40.0 mm to (131.8, 55.0)
- moved R35 40.0 mm to (133.2, 55.0)
- moved R36 40.0 mm to (134.8, 55.0)
- moved R37 40.0 mm to (136.2, 55.0)
- moved R38 40.0 mm to (137.8, 55.0)
- moved R39 40.0 mm to (139.2, 55.0)
- moved R40 40.0 mm to (140.8, 55.0)
- moved R41 40.0 mm to (142.2, 55.0)
- moved R42 40.0 mm to (143.8, 55.0)
- moved R43 40.0 mm to (145.2, 55.0)
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Connections:
- J15 pad 2: SND -> CASSETTE_OUT
- U1 pad 18: USB_DM1 -> AUDIO_R
- U1 pad 20: USB_DP1 -> AUDIO_L
- U1 pad 21: USB_DM2 -> CASSETTE_OUT
- U1 pad 23: USB_DP2 -> CASSETTE_IN
- U1 pad 24: AUDIO_R -> PRINTER_IN
- U1 pad 25: AUDIO_L -> PRINTER_OUT
- U1 pad 31: CASSETTE_OUT -> ESP_NOTIFY
- U1 pad 32: CASSETTE_IN -> USB_DM2
- U1 pad 33: PRINTER_IN -> USB_DP2
- U1 pad 35: PRINTER_OUT -> USB_DM1
- U1 pad 36: ESP_NOTIFY -> USB_DP1
- U5 pad 10: ESP_NOTIFY -> SD_SSEL#
- U5 pad 12: unconnected-(U5-Pad12) -> FPGA_DONE
- U5 pad 15: unconnected-(U5-Pad15) -> SPI_MISO
- U5 pad 17: ESP_TX -> SPI_MOSI
- U5 pad 18: ESP_RTS -> SPI_SCLK
- U5 pad 19: ESP_RX -> SPI_CS#
- U5 pad 20: ESP_CTS -> ESP_NOTIFY
- U5 pad 21: SD_MISO -> ESP_TX
- U5 pad 22: SD_MOSI -> ESP_RTS
- U5 pad 23: SD_SCK -> ESP_RX
- U5 pad 24: SD_SSEL# -> ESP_CTS
- U5 pad 25: SD_WP# -> FPGA_PROG#
- U5 pad 28: SD_CD# -> unconnected-(U5-Pad28)
- U5 pad 29: SD_ACTIVITY -> unconnected-(U5-Pad29)
- U5 pad 4: SPI_CS# -> SD_ACTIVITY
- U5 pad 5: SPI_SCLK -> SD_WP#
- U5 pad 6: SPI_MOSI -> SD_CD#
- U5 pad 7: SPI_MISO -> SD_MISO
- U5 pad 8: FPGA_PROG# -> SD_SCK
- U5 pad 9: FPGA_DONE -> SD_MOSI
Routing:
- net +5V: track 2.68 -> 316.7 mm, vias 1 -> 7
- net CASSETTE_OUT: track 0.00 -> 190.9 mm, vias 0 -> 4
- net +3V3: track 133.2 -> 249.4 mm, vias 21 -> 27
- net CART_CE#: track 0.00 -> 115.6 mm, vias 0 -> 2
- net BUSREQ#: track 0.00 -> 111.1 mm, vias 0 -> 4
- net RESET#: track 0.00 -> 109.3 mm, vias 0 -> 6
- net INT#: track 0.00 -> 106.9 mm, vias 0 -> 2
- net M1#: track 0.00 -> 98.4 mm, vias 0 -> 4
- net A13: track 34.1 -> 124.5 mm, vias 1 -> 6
- net A3: track 28.9 -> 115.6 mm, vias 1 -> 9
- net WR#: track 35.5 -> 121.6 mm, vias 1 -> 4
- net A10: track 27.3 -> 111.6 mm, vias 1 -> 9
- net ESP_USB_DM: track 0.00 -> 83.7 mm
- net A11: track 30.3 -> 111.8 mm, vias 1 -> 9
- net A12: track 35.6 -> 116.2 mm, vias 1 -> 4
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