File: pcb/aquarius-plus.kicad_sch (KiCad schematic)
At the start: 23 parts

Commit message: Working on schematic.
Parts:
- removed R? (x2): (no value), symbol Device:R
- removed R?: 4.7k, symbol Device:R
- removed R? (x2): 220, symbol Device:R
- added C? (x3): 100nF, symbol Device:C_Small
- added C? (x7): (no value), symbol Device:C_Small
- added C?: 10uF, symbol Device:C_Small
- added C?: (no value), symbol Device:C
- added D?: 1N4148W, Diode_SMD:D_SOD-123, symbol Diode:1N4148W
- added D?: (no value), symbol Diode:1N4148W
- added D? (x2): (no value), symbol Device:LED
- added J? (x4): (no value), symbol Connector:AudioJack3
- added J? (x2): (no value), symbol Connector:DB9_Male_MountingHoles
- added J?: (no value), symbol Connector:SD_Card
- added J? (x2): USB_A, symbol Connector:USB_A
- added J?: (no value), symbol Connector:USB_A
- added J?: (no value), symbol Connector:DB15_Female_HighDensity_MountingHoles
- added J?: (no value), symbol Connector:USB_B_Micro
- added J?: (no value), symbol Connector:Conn_Coaxial
- added J?: (no value), symbol Connector_Generic:Conn_01x03
- added JP? (x3): (no value), symbol Jumper:Jumper_2_Open
- added Q?: (no value), Package_TO_SOT_SMD:SOT-23, symbol Transistor_BJT:BC847
- added Q?: (no value), symbol Transistor_BJT:BC847
- added R? (x3): 33, symbol Device:R
- added R? (x2): 4.7k, symbol Device:R
- added R? (x38): (no value), symbol Device:R
- added R? (x33): 100, symbol Device:R
- added R? (x2): 536, symbol Device:R
- added R? (x2): 220, symbol Device:R
- added R? (x3): 15k, symbol Device:R
- added R?: 150, symbol Device:R
- added R? (x2): 2150, symbol Device:R
- added R? (x2): 1070, symbol Device:R
- added R? (x2): 4300, symbol Device:R
- added R?: 330, symbol Device:R
- added R?: 1k, symbol Device:R
- added SW? (x2): (no value), symbol Switch:SW_DPDT_x2
- added U?: ESP32-S2-SOLO-N4R2, symbol aquarius-plus:ESP32-S2-SOLO-N4R2
- added U?: (no value), symbol Interface_UART:MAX3221
- added U? (x3): SN74CBTD3861PWR, Package_SO:TSSOP-24_4.4x7.8mm_P0.65mm, symbol 74xx:74CBTLV3861
- added U? (x2): (no value), symbol 74xx:74LS166
- added U?: (no value), symbol Logic_LevelTranslator:SN74AVC8T245PW
- added U?: (no value), symbol 74xx:74CBTLV3861
- added X?: SG-5032CAN, Oscillator:Oscillator_SMD_SeikoEpson_SG8002LB-4Pin_5.0x3.2mm, symbol Oscillator:SG-5032CAN
- J?: value (none) -> Expansion port
- R?: value (none) -> 220
- R?: value (none) -> DNP
- R?: value (none) -> 1k
- U?: value (none) -> XC3S200-4TQG144; footprint (none) -> Package_QFP:TQFP-144_20x20mm_P0.5mm
- U?: value (none) -> Z84C0010AEG
- U?: value (none) -> IS61C5128AS-25QLI
- U?: value (none) -> SST39SF020A-55-4C-WHE
- X?: value (none) -> SG-5032CAN
Connections:
- net +3V3: now also C?.1, J?.4 (VDD), R?.1, R?.2, R?.2, R?.2, R?.2, R?.2, R?.2, R?.2, R?.2, R?.2, R?.2, R?.2, R?.2, R?.2, R?.2, R?.2, R?.2, R?.2, R?.2, R?.2, R?.2, R?.2, R?.2, R?.2, R?.2, R?.2, R?.2, R?.2, R?.2, U?.1 (VCCA), U?.12 (FORCEON), U?.15 (VCC), U?.16 (VCC), U?.16 (VCC), U?.16 (~{FORCEOFF}), U?.2 (3V3), U?.9 (Clr), U?.9 (Clr), X?.4 (VCC)
- net +5V: now also J?.1 (VBUS), J?.1 (VBUS), J?.1 (VBUS), R?.1, SW?.1 (A), SW?.4 (A), U?.23 (VCCB), U?.24 (VCC), U?.24 (VCC), U?.24 (VCC), U?.24 (VCC), U?.24 (VCCB)
- net A0: now also U?.22 (B1)
- net A1: now also U?.21 (B2)
- net A10: now also U?.22 (B1)
- net A11: now also U?.21 (B2)
- net A12: now also U?.20 (B3)
- net A13: now also U?.19 (B4)
- net A14: now also U?.18 (B5)
- net A15: now also U?.17 (B6)
- net A2: now also U?.20 (B3)
- net A3: now also U?.19 (B4)
- net A4: now also U?.18 (B5)
- net A5: now also U?.17 (B6)
- net A6: now also U?.16 (B7)
- net A7: now also U?.15 (B8)
- net A8: now also U?.14 (B9)
- net A9: now also U?.13 (B10)
- net AUDIO_L: now also U?.25 (B6_IO), R?.1
- net AUDIO_R: now also U?.24 (B6_IO_VREF), R?.1
- net BA14: now also U?.122 (B1_IO)
- net BA15: now also U?.125 (B1_IO_GCLK5)
- net BA16: now also U?.124 (B1_IO_GCLK4)
- net BA17: now also U?.108 (B2_IO)
- net BA18: now also U?.107 (B2_IO)
- net BUSACK#: now also U?.20 (B3)
- net BUSREQ#: now also U?.21 (B2)
- net CASSETTE_IN: now also U?.32 (B6_IO), Q?.3 (C), R?.1
- net D0: now also U?.16 (B7)
- net D1: now also U?.15 (B8)
- net D2: now also U?.14 (B9)
- net D3: now also U?.13 (B10)
- net D4: now also U?.22 (B1)
- net D5: now also U?.21 (B2)
- net D6: now also U?.20 (B3)
- net D7: now also U?.19 (B4)
- net DE0: now also U?.21 (B1)
- net DE1: now also U?.20 (B2)
- net DE2: now also U?.19 (B3)
- net DE3: now also U?.18 (B4)
- net DE4: now also U?.17 (B5)
- net DE5: now also U?.16 (B6)
- net DE6: now also U?.15 (B7)
- net DE7: now also U?.14 (B8)
- net ESP_CTS: now also U?.26 (B6_IO), U?.20 (IO12)
- net ESP_RTS: now also U?.28 (B6_IO), U?.18 (IO10)
- net ESP_RX: now also U?.27 (B6_IO), U?.19 (IO11)
- net ESP_TX: now also U?.30 (B6_IO), U?.17 (IO9)
- net FPGA_DONE: now also R?.1, U?.9 (IO16)
- net FPGA_PROG#: now also R?.1, U?.8 (IO15)
- net GND: now also C?.2, C?.2, C?.2, C?.2, C?.2, C?.2, D?.1 (K), D?.1 (K), D?.2 (A), D?.2 (A), J?.0, J?.0 (PAD), J?.0 (PAD), J?.1, J?.1, J?.10, J?.12 (SHELL1), J?.13 (SHELL2), J?.2 (Ext), J?.3 (Pin_3), J?.3 (VSS), J?.4 (GND), J?.4 (GND), J?.4 (GND), J?.5, J?.5 (GND), J?.5 (Shield), J?.5 (Shield), J?.5 (Shield), J?.6, J?.6 (Shield), J?.6 (VSS), J?.7, J?.8, J?.S, J?.S, J?.S, J?.S, JP?.2 (B), Q?.2 (E), R?.1, R?.1, R?.1, R?.1, R?.1, R?.2, R?.2, R?.2, R?.2, U?.1 (Ds), U?.1 (GND), U?.1 (~{EN}), U?.11 (GND), U?.12 (GND), U?.12 (GND), U?.12 (GND), U?.12 (GND), U?.12 (GND), U?.13 (GND), U?.14 (GND), U?.23 (OE), U?.23 (OE), U?.23 (OE), U?.23 (OE), U?.40 (GND), U?.41 (EPAD), U?.6 (CE), U?.6 (CE), U?.8 (GND), U?.8 (GND), X?.2 (GND)
- net INT#: now also U?.22 (B1)
- net IORQ#: now also U?.16 (B7)
- net M1#: now also U?.18 (B5)
- net MREQ#: now also U?.17 (B6)
- net PRINTER_IN: now also U?.33 (B6_IO), U?.9 (ROUT)
- net PRINTER_OUT: now also U?.35 (B6_IO), U?.11 (DIN)
- net RAM_CE#: now also U?.79 (B3_IO)
- net RD#: now also U?.15 (B8), U?.2 (DIR)
- net RESET#: now also U?.19 (B4)
- net ROM_CE#: now also U?.83 (B3_IO)
- net SPI_CS#: now also R?.1, U?.4 (IO4)
- net SPI_MISO: now also U?.7 (IO7)
- net SPI_MOSI: now also U?.6 (IO6)
- net SPI_SCLK: now also U?.5 (IO5)
- net SYSCLK: now also U?.55 (B4_IO_GCLK0)
- net USB_DM1: now also U?.15 (B7_IO), R?.1, R?.2
- net USB_DM2: now also U?.18 (B7_IO_VREF), R?.1, R?.2
- net USB_DP1: now also U?.14 (B7_IO), R?.1, R?.2
- net USB_DP2: now also U?.17 (B7_IO), R?.1, R?.2
- net VGA_B0: now also U?.8 (B7_IO), R?.1
- net VGA_B1: now also U?.7 (B7_IO), R?.1
- net VGA_B2: now also U?.11 (B7_IO), R?.1
- net VGA_B3: now also U?.10 (B7_IO), R?.1
- net VGA_G0: now also U?.2 (B7_IO), R?.1
- net VGA_G1: now also U?.1 (B7_IO), R?.1
- net VGA_G2: now also U?.6 (B7_IO), R?.1
- net VGA_G3: now also U?.5 (B7_IO), R?.1
- net VGA_HSYNC: now also U?.13 (B7_IO), R?.1
- net VGA_R0: now also U?.23 (B6_IO), R?.1
- net VGA_R1: now also U?.21 (B6_IO), R?.1
- net VGA_R2: now also U?.20 (B6_IO_VREF), R?.1
- net VGA_R3: now also U?.4 (B7_IO_VREF), R?.1
- net VGA_VSYNC: now also U?.12 (B7_IO), R?.1
- net WAIT#: now also U?.13 (B10)
- net WR#: now also U?.14 (B9)
- net FPGA_D4: now reaches U?.100 (B2_IO)
- net FPGA_D4: now also U?.2 (A1)
- net FPGA_D3: now reaches U?.102 (B2_IO)
- net FPGA_D3: now also U?.11 (A10)
- net FPGA_D2: now reaches U?.103 (B2_IO)
- net FPGA_D2: now also U?.10 (A9)
- net FPGA_D1: now reaches U?.104 (B2_IO)
- net FPGA_D1: now also U?.9 (A8)
- net FPGA_D0: now reaches U?.105 (B2_IO)
- net FPGA_D0: now also U?.8 (A7)
- net FPGA_A12: now reaches U?.112 (B1_IO)
- net FPGA_A12: now also U?.4 (A3)
- net FPGA_A11: now reaches U?.113 (B1_IO)
- net FPGA_A11: now also U?.3 (A2)
- net FPGA_A10: now reaches U?.116 (B1_IO)
- net FPGA_A10: now also U?.2 (A1)
- net FPGA_A14: now reaches U?.118 (B1_IO)
- net FPGA_A14: now also U?.6 (A5)
- net FPGA_A13: now reaches U?.119 (B1_IO)
- net FPGA_A13: now also U?.5 (A4)
- net FPGA_A15: now reaches U?.123 (B1_IO_VREF)
- net FPGA_A15: now also U?.7 (A6)
- net FPGA_A9: now reaches U?.127 (B0_IO_GCLK6)
- net FPGA_A9: now also U?.11 (A10)
- net FPGA_A8: now reaches U?.128 (B0_IO_GCLK7)
- net FPGA_A8: now also U?.10 (A9)
- net FPGA_A7: now reaches U?.129 (B0_IO_VREF)
- net FPGA_A7: now also U?.9 (A8)
- net FPGA_A6: now reaches U?.130 (B0_IO)
- net FPGA_A6: now also U?.8 (A7)
- net FPGA_A5: now reaches U?.131 (B0_IO)
- net FPGA_A5: now also U?.7 (A6)
- net FPGA_A4: now reaches U?.132 (B0_IO)
- net FPGA_A4: now also U?.6 (A5)
- net FPGA_A3: now reaches U?.135 (B0_IO)
- net FPGA_A3: now also U?.5 (A4)
- net FPGA_A2: now reaches U?.137 (B0_IO)
- net FPGA_A2: now also U?.4 (A3)
- net FPGA_A1: now reaches U?.140 (B0_IO)
- net FPGA_A1: now also U?.3 (A2)
- net FPGA_A0: now reaches U?.141 (B0_IO)
- net FPGA_A0: now also U?.2 (A1)
- net at U?.143 (PROG_B): now also R?.1, R?.2
- net CASSETTE_OUT: now reaches U?.31 (B6_IO)
- net CASSETTE_OUT: now also R?.1
- net ESP_NOTIFY: now reaches U?.36 (B6_IO)
- net ESP_NOTIFY: now also U?.10 (IO17)
- net CVID3: now reaches U?.40 (B5_IO)
- net CVID3: now also R?.1
- net CVID4: now reaches U?.41 (B5_IO)
- net CVID4: now also R?.1
- net CVID5: now reaches U?.44 (B5_IO_VREF)
- net CVID5: now also R?.1
- net CVID1: now reaches U?.46 (B5_IO)
- net CVID1: now also R?.1
- net CVID2: now reaches U?.47 (B5_IO)
- net CVID2: now also R?.1
- net CVID0: now reaches U?.51 (B5_IO)
- net CVID0: now also R?.1
- net USBCLK: now reaches U?.52 (B5_IO_GCLK2)
- net USBCLK: now also X?.3 (OUT)
- net HCTRL_DATA: now reaches U?.56 (B4_IO_GCLK1)
- net HCTRL_DATA: now also U?.13 (Qh)
- net at U?.58 (B4_IO_INIT_B): now also R?.1, R?.2
- net HCTRL_LOAD#: now reaches U?.59 (B4_IO)
- net HCTRL_LOAD#: now also U?.15 (PE), U?.15 (PE)
- net HCTRL_CLK: now reaches U?.60 (B4_IO)
- net HCTRL_CLK: now also U?.7 (Clk), U?.7 (Clk)
- net DE_OE#: now reaches U?.63 (B4_IO)
- net DE_OE#: now also U?.22 (~{OE})
- net FPGA_DE7: now reaches U?.68 (B4_IO)
- net FPGA_DE7: now also U?.10 (A8)
- net FPGA_DE6: now reaches U?.69 (B4_IO)
- net FPGA_DE6: now also U?.9 (A7)
- net FPGA_DE5: now reaches U?.70 (B4_IO_VREF)
- net FPGA_DE5: now also U?.8 (A6)
- net FPGA_INT#: now reaches U?.73 (B3_IO)
- net FPGA_INT#: now also U?.2 (A1)
- net FPGA_WAIT#: now reaches U?.74 (B3_IO)
- net FPGA_WAIT#: now also U?.11 (A10)
- net FPGA_WR#: now reaches U?.76 (B3_IO)
- net FPGA_WR#: now also U?.10 (A9)
- net FPGA_BUSREQ#: now reaches U?.77 (B3_IO)
- net FPGA_BUSREQ#: now also U?.3 (A2)
- net FPGA_RESET#: now reaches U?.78 (B3_IO)
- net FPGA_RESET#: now also U?.5 (A4)
- net FPGA_BUSACK#: now reaches U?.80 (B3_IO)
- net FPGA_BUSACK#: now also U?.4 (A3)
- net FPGA_DE0: now reaches U?.84 (B3_IO_VREF)
- net FPGA_DE0: now also U?.3 (A1)
- net FPGA_DE2: now reaches U?.86 (B3_IO)
- net FPGA_DE2: now also U?.5 (A3)
- net FPGA_DE1: now reaches U?.87 (B3_IO)
- net FPGA_DE1: now also U?.4 (A2)
- net FPGA_DE4: now reaches U?.89 (B3_IO)
- net FPGA_DE4: now also U?.7 (A5)
- net FPGA_DE3: now reaches U?.90 (B3_IO_VREF)
- net FPGA_DE3: now also U?.6 (A4)
- net FPGA_RD#: now reaches U?.92 (B2_IO_VREF)
- net FPGA_RD#: now also U?.9 (A8)
- net FPGA_IORQ#: now reaches U?.93 (B2_IO)
- net FPGA_IORQ#: now also U?.8 (A7)
- net FPGA_MREQ#: now reaches U?.95 (B2_IO)
- net FPGA_MREQ#: now also U?.7 (A6)
- net FPGA_M1#: now reaches U?.96 (B2_IO)
- net FPGA_M1#: now also U?.6 (A5)
- net FPGA_D7: now reaches U?.97 (B2_IO)
- net FPGA_D7: now also U?.5 (A4)
- net FPGA_D6: now reaches U?.98 (B2_IO_VREF)
- net FPGA_D6: now also U?.4 (A3)
- net FPGA_D5: now reaches U?.99 (B2_IO)
- net FPGA_D5: now also U?.3 (A2)
- net CSYNC#: no longer names the net of J?.1 (Pin_1)
- new net: J?.R, U?.8 (RIN)
- new net: J?.T, U?.13 (DOUT)
- new net: D?.1 (K), Q?.1 (B), R?.1, R?.2
- new net: J?.3 (D+), R?.1 (x2)
- new net: J?.5 (CLK), R?.2
- new net: R?.1, R?.2, U?.5 (D) (x2)
- new net: J?.T, R?.1
- new net: C?.1, R?.2, R?.2
- new net: J?.2, R?.2, R?.2, R?.2, R?.2
- new net: J?.3, R?.1 (x2)
- new net: R?.1, R?.2, U?.10 (E) (x2)
- new net: J?.2, R?.1 (x2)
- new net: R?.1, R?.2, U?.12 (G) (x2)
- new net: J?.4, R?.1 (x2)
- new net: J?.5, R?.1 (x2)
- new net: J?.6, R?.1 (x2)
- new net: J?.7, R?.1 (x2)
- new net: J?.8, R?.1 (x2)
- new net: J?.9, R?.1 (x2)
- new net: J?.2 (D-), JP?.1 (A)
- new net: J?.1 (CD/DAT3), R?.2
- new net: J?.2 (CMD), R?.2
- new net: J?.7 (DAT0), R?.2
- new net: J?.8 (DAT1), R?.1
- new net: J?.9 (DAT2), R?.1
- new net: JP?.1 (A), U?.27 (IO0)
- new net: C?.1, R?.2, U?.3 (EN)
- new net: J?.2 (Pin_2), U?.36 (IO44/RXD0)
- new net: J?.1 (Pin_1), U?.37 (IO32/TXD0)
- new net: C?.1, U?.2 (C1+)
- new net: C?.2, U?.4 (C1-)
- new net: C?.1, U?.3 (V+)
- new net: C?.1, U?.5 (C2+)
- new net: C?.2, U?.6 (C2-)
- new net: C?.1, U?.7 (V-)
- new net: R?.1, R?.2, U?.3 (B) (x2)
- new net: R?.1, R?.2, U?.4 (C) (x2)
- new net: R?.1, R?.2, U?.11 (F) (x2)
- new net: R?.1, R?.2, U?.2 (A) (x2)
- new net: R?.1, R?.2, U?.14 (H) (x2)
- new net: J?.3, R?.2, R?.2, R?.2, R?.2
- new net: J?.R, J?.T, R?.2, R?.2
- new net: J?.2 (D-), R?.1 (x2)
- new net: J?.R, R?.1
- new net: Q?.2 (E), R?.2
- new net: C?.1, Q?.3 (C), R?.1
- new net: C?.2, R?.1
- new net: J?.1 (In), R?.2, R?.2, R?.2, R?.2, R?.2, R?.2
- new net: C?.1, C?.1, R?.2, R?.2 (x2)
- new net: J?.1, R?.2, R?.2, R?.2, R?.2
- new net: C?.2, D?.1 (K), Q?.1 (B), R?.1, R?.2
- new net: J?.13, R?.2
- new net: J?.14, R?.2
- new net: C?.2, J?.R
- new net: J?.3 (D+), JP?.1 (A)
- new net: D?.2 (A), R?.2 (x2)
- new net: C?.2, J?.T
- new net: U?.1 (Ds), U?.13 (Qh)
- new net ESP_USB_DM: J?.2 (D-), JP?.2 (B), U?.13 (IO19/USB_DM)
- new net ESP_USB_DP: J?.3 (D+), JP?.2 (B), U?.14 (IO20/USB_DP)
- new net SD_ACTIVITY: R?.1, U?.29 (IO36)
- new net SD_CD#: J?.10 (CARD_DETECT), U?.28 (IO35)
- new net SD_MISO: R?.1, R?.1, U?.21 (IO13)
- new net SD_MOSI: R?.1, R?.1, U?.22 (IO14)
- new net SD_SCK: R?.1, U?.23 (IO21)
- new net SD_SSEL#: R?.1, R?.1, U?.24 (IO33)
- new net SD_WP#: J?.11 (WRITE_PROTECT), U?.25 (IO34)
- new net VBUS: J?.1 (VBUS), SW?.2 (B), SW?.5 (B)
- no-connect marks 1 -> 14
Other:
- note added: "256KB Flash"
- note added: "512KB SRAM"
- note added: "Audio output"
- note added: "Cartridge port"
- note added: "Cassette interface"
- note added: "Composite video output"
- note added: "ESP32"
- note added: "Ext. data bus level translation"
- note added: "FPGA"
- note added: "Handcontroller interface"
- note added: "LEDs"
- note added: "Level translation"
- note added: "Power switch"
- note added: "Secure Digital card interface"
- note added: "Serial printer port"
- note added: "System clock (14.31818MHz)"
- note added: "USB clock (48MHz)"
- note added: "USB host / slave via ESP32"
- note added: "USB host via FPGA"
- note added: "VGA interface"
- note added: "Various pullups"
- note added: "Z80 processor"
- moved on the sheet: J?, R?, U?, X?

Commit message: Worked on schematic.
Parts:
- removed C?: (no value), symbol Device:C
- added C? (x34): 100nF, symbol Device:C_Small
- added C? (x10): 4.7uF, symbol Device:C_Small
- added C? (x8): (no value), symbol Device:C_Small
- added C? (x3): 100uF, symbol Device:C_Polarized_Small
- added C?: (no value), symbol Device:C_Polarized_Small
- added R? (x2): (no value), symbol Device:R
- added R? (x2): 1, symbol Device:R
- added U?: 74LVC4245APW, Package_SO:TSSOP-24_4.4x7.8mm_P0.65mm, symbol Logic_LevelTranslator:SN74AVC8T245PW
- added U?: (no value), Package_TO_SOT_SMD:SOT-223-3_TabPin2, symbol Regulator_Linear:AP1117-33
- added U?: (no value), symbol Regulator_Linear:AP1117-33
- added U?: (no value), symbol Regulator_Linear:MCP1700-2502E_SOT23
- C?: value (none) -> 1uF
- C?: value (none) -> 4.7uF
- C? (x4): value (none) -> 100nF
- C?: value (none) -> 10uF
- D?: value (none) -> 1N4148W; footprint (none) -> Diode_SMD:D_SOD-123
- D?: value (none) -> SD act.
- D?: value (none) -> Power
- J?: value (none) -> Printer
- J?: value (none) -> Hand controller 1
- J?: value (none) -> SD_Card
- J?: value (none) -> Cassette out
- J?: value (none) -> ESP USB Host
- J?: value (none) -> VGA
- J?: value (none) -> Cassette in
- J?: value (none) -> Audio out
- J?: value (none) -> Power in
- J?: value (none) -> Composite
- J?: value (none) -> Hand controller 2
- J?: value (none) -> DBG
- JP? (x2): value (none) -> USB
- JP?: value (none) -> Bootloader
- Q?: value (none) -> BC847C
- Q?: value (none) -> BC847C; footprint (none) -> Package_TO_SOT_SMD:SOT-23
- R? (x7): value (none) -> 10k
- R? (x4): value (none) -> 4.7k
- R?: value (none) -> 15k
- R? (x4): value (none) -> 100
- R? (x2): value (none) -> 220
- R?: value (none) -> 33
- R? (x6): value (none) -> TBD
- R?: value (none) -> 330
- R?: value (none) -> 2150
- R?: value (none) -> 1070
- R?: value (none) -> 4300
- R? (x2): value (none) -> 47k
- R?: value (none) -> 536
- R? (x2): value (none) -> 820
- R?: value (none) -> 220k
- R?: value (none) -> 470
- R?: value (none) -> 2.2k
- R?: value (none) -> 150
- SW? (x2): value (none) -> SW_DPDT_x2
- U?: value (none) -> MAX3221
- U? (x2): value (none) -> 74HC166
- U?: value (none) -> 74LVC4245APW; footprint (none) -> Package_SO:TSSOP-24_4.4x7.8mm_P0.65mm
- U?: value (none) -> SN74CBTD3861PWR; footprint (none) -> Package_SO:TSSOP-24_4.4x7.8mm_P0.65mm
Connections:
- net +1V2: now also C?.1, C?.1, C?.1, C?.1, C?.1, C?.1, C?.1, R?.2, U?.2 (VO)
- net +2V5: now also C?.1, C?.1, C?.1, C?.1, C?.1, C?.1, C?.1, U?.2 (VO)
- net +3V3: now also C?.1, C?.1, C?.1, C?.1, C?.1, C?.1, C?.1, C?.1, C?.1, C?.1, C?.1, C?.1, C?.1, C?.1, C?.1, C?.1, C?.1, C?.1, C?.1, C?.1, C?.1, C?.1, C?.1, C?.1, C?.1, R?.1, R?.1, U?.2 (VO), U?.23 (VCCB), U?.24 (VCCB)
- net +5V: now also C?.1, C?.1, C?.1, C?.1, C?.1, C?.1, C?.1, C?.1, C?.1, C?.1, C?.1, C?.1, C?.1, R?.1, U?.1 (VCCA)
- net CART_CE#: now also U?.4 (A2)
- net GND: now also C?.2, C?.2, C?.2, C?.2, C?.2, C?.2, C?.2, C?.2, C?.2, C?.2, C?.2, C?.2, C?.2, C?.2, C?.2, C?.2, C?.2, C?.2, C?.2, C?.2, C?.2, C?.2, C?.2, C?.2, C?.2, C?.2, C?.2, C?.2, C?.2, C?.2, C?.2, C?.2, C?.2, C?.2, C?.2, C?.2, C?.2, C?.2, C?.2, C?.2, C?.2, C?.2, C?.2, C?.2, C?.2, C?.2, C?.2, C?.2, C?.2, C?.2, C?.2, C?.2, C?.2, C?.2, C?.2, C?.2, R?.1, U?.1 (GND), U?.1 (GND), U?.1 (GND), U?.11 (GND), U?.12 (GND), U?.13 (GND), U?.2 (DIR), U?.22 (~{OE})
- net PHI: now also U?.3 (A1)
- net FPGA_PHI: now reaches U?.82 (B3_IO)
- net FPGA_PHI: now also U?.21 (B1)
- net FPGA_CART_CE#: now reaches U?.85 (B3_IO)
- net FPGA_CART_CE#: now also U?.20 (B2)
- net at R?.2, U?.3 (EN): now also C?.1
- new net: C?.1, R?.2, U?.3 (VI) (x3)
Other:
- note added: "Power supply"
- note removed: "Ext. data bus level translation"
- note removed: "Power switch"
- company: (none) -> Designed by Frank van den Hoef
- title: (none) -> Aquarius+
- moved on the sheet: C?, D?, J?, JP?, Q?, R?, SW?A, SW?B, U?, X?

Commit message: Working on PCB layout.
Parts:
- removed D? (x2): 1N4148W, Diode_SMD:D_SOD-123, symbol Diode:1N4148W
- removed D?: Power, symbol Device:LED
- removed J?: Composite, symbol Connector:Conn_Coaxial
- removed R? (x6): TBD, symbol Device:R
- removed R?: 470, symbol Device:R
- added D1, D2: 1N4148WS, Diode_SMD:D_SOD-323_HandSoldering, symbol Diode:1N4148WS
- added H1, H2, H3, H4: MountingHole, MountingHole:MountingHole_3.2mm_M3, symbol Mechanical:MountingHole
- added J14: FPGA spare, Connector_PinHeader_2.54mm:PinHeader_2x05_P2.54mm_Vertical, symbol Connector_Generic:Conn_02x05_Odd_Even
- added J16: ESP32 spare, Connector_PinHeader_2.54mm:PinHeader_2x05_P2.54mm_Vertical, symbol Connector_Generic:Conn_02x05_Odd_Even
- C1, C36: renamed from C?; value (none) -> 100nF; footprint (none) -> Capacitor_SMD:C_0603_1608Metric
- C10, C15, C20, C21, C5: renamed from C?; value (none) -> 4.7uF; footprint (none) -> Capacitor_SMD:C_0603_1608Metric
- C11, C12, C13, C14, C16, C17, C18, C19, C2, C22, C23, C24, C25, C26, C27, C28, C29, C3, C30, C31, C32, C33, C34, C35, C38, C39, C4, C41, C42, C43, C44, C45, C46, C50, C51, C52, C55, C56, C57, C58, C59, C6, C60, C62, C63, C64, C65, C66, C67, C7, C8, C9: renamed from C?; footprint (none) -> Capacitor_SMD:C_0603_1608Metric
- C37: renamed from C?; value (none) -> 22uF; footprint (none) -> Capacitor_SMD:C_1206_3216Metric
- C40: renamed from C?; value 1uF -> 4.7uF; footprint (none) -> Capacitor_SMD:C_0603_1608Metric
- C47, C53, C54: renamed from C?; footprint (none) -> Capacitor_SMD:CP_Elec_6.3x7.7
- C48, C49: renamed from C?; footprint (none) -> Capacitor_SMD:C_0805_2012Metric
- C61: renamed from C?; value (none) -> 100uF; footprint (none) -> Capacitor_SMD:CP_Elec_6.3x7.7
- D4: renamed from D?; footprint (none) -> LED_THT:LED_D3.0mm_Horizontal_O1.27mm_Z2.0mm
- J1, J10, J2, J4: renamed from J?; footprint (none) -> Connector_Audio:Jack_3.5mm_CUI_SJ-3523-SMT_Horizontal
- J11, J5: renamed from J?; footprint (none) -> Connector_Dsub:DSUB-9_Male_Horizontal_P2.77x2.84mm_EdgePinOffset9.90mm_Housed_MountingHolesOffset11.32mm
- J12, J8, J9: renamed from J?; footprint (none) -> Connector_USB:USB_A_Molex_67643_Horizontal
- J13: renamed from J?; footprint (none) -> aquarius-plus:10118193-0001LF
- J15: renamed from J?; footprint (none) -> aquarius-plus:CR22A-44D-2.54DSA(70)
- J3: renamed from J?; footprint (none) -> Connector_Card:SD_TE_2041021
- J6: renamed from J?; footprint (none) -> aquarius-plus:ICD15S13E4GV00LF
- J7: renamed from J?; footprint (none) -> Connector_PinHeader_2.54mm:PinHeader_1x03_P2.54mm_Vertical
- JP1, JP2, JP3: renamed from JP?; footprint (none) -> Connector_PinHeader_2.54mm:PinHeader_1x02_P2.54mm_Vertical
- R1, R10, R100, R101, R11, R12, R13, R14, R15, R16, R17, R18, R19, R2, R20, R21, R22, R23, R24, R25, R26, R27, R28, R29, R3, R30, R31, R32, R33, R34, R35, R36, R37, R38, R39, R4, R40, R41, R42, R43, R44, R45, R46, R47, R48, R49, R5, R50, R51, R52, R54, R55, R56, R57, R58, R59, R6, R60, R61, R62, R7, R71, R72, R73, R74, R75, R76, R77, R78, R79, R8, R80, R81, R82, R83, R84, R85, R86, R87, R88, R89, R9, R90: renamed from R?; footprint (none) -> Resistor_SMD:R_0603_1608Metric
- R102: renamed from R?; value (none) -> 100; footprint (none) -> Resistor_SMD:R_0603_1608Metric
- R63, R64, R65, R66, R67, R68, R69, R70, R91, R92, R93, R94, R95, R96, R97, R98: renamed from R?; value 100 -> 4.7k; footprint (none) -> Resistor_SMD:R_0603_1608Metric
- R99: renamed from R?; value (none) -> 1; footprint (none) -> Resistor_SMD:R_0603_1608Metric
- SW1: renamed from SW?; footprint (none) -> Button_Switch_THT:SW_E-Switch_EG2219_DPDT_Angled
- U12, U9: renamed from U?; footprint (none) -> Package_SO:SOIC-16_3.9x9.9mm_P1.27mm
- U15: renamed from U?; value (none) -> LDL1117S33R; footprint (none) -> Package_TO_SOT_SMD:SOT-223-3_TabPin2
- U16: renamed from U?; value (none) -> MCP1700T-2502E/TT; footprint (none) -> Package_TO_SOT_SMD:SOT-23
- U17: renamed from U?; value (none) -> LD1117S12
- U3: renamed from U?; value MAX3221 -> MAX3221ECPWR; footprint (none) -> Package_SO:TSSOP-16_4.4x5mm_P0.65mm
- U5: renamed from U?; footprint (none) -> aquarius-plus:ESP32-S2-SOLO-N4R2
- gave numbers to parts that had none: 14
Connections:
- net +3V3: now also U14.1 (VCCA), U14.2 (DIR), J14.1 (Pin_1), J16.1 (Pin_1); no longer U14.23 (VCCB), U14.24 (VCCB)
- net +5V: now also J9.1 (VBUS), U14.23 (VCCB), U14.24 (VCCB); no longer J13.1 (VBUS), U14.1 (VCCA)
- net A0: now also U2.16 (B7); no longer U2.22 (B1)
- net A1: now also U2.15 (B8); no longer U2.21 (B2)
- net A10: now also U8.16 (B7); no longer U4.22 (B1)
- net A11: now also U8.15 (B8); no longer U4.21 (B2)
- net A12: now also U8.14 (B9); no longer U4.20 (B3)
- net A13: now also U8.13 (B10); no longer U4.19 (B4)
- net A14: now also U4.22 (B1); no longer U4.18 (B5)
- net A15: now also U4.21 (B2); no longer U4.17 (B6)
- net A2: now also U2.14 (B9); no longer U2.20 (B3)
- net A3: now also U2.13 (B10); no longer U2.19 (B4)
- net A4: now also U8.22 (B1); no longer U2.18 (B5)
- net A5: now also U8.21 (B2); no longer U2.17 (B6)
- net A6: now also U8.20 (B3); no longer U2.16 (B7)
- net A7: now also U8.19 (B4); no longer U2.15 (B8)
- net A8: now also U8.18 (B5); no longer U2.14 (B9)
- net A9: now also U8.17 (B6); no longer U2.13 (B10)
- net BA14: now also U1.141 (B0_IO); no longer U1.122 (B1_IO)
- net BA15: now also U1.140 (B0_IO); no longer U1.125 (B1_IO_GCLK5)
- net BA16: now also U1.137 (B0_IO); no longer U1.124 (B1_IO_GCLK4)
- net BA17: now also U1.135 (B0_IO); no longer U1.108 (B2_IO)
- net BA18: now also U1.132 (B0_IO); no longer U1.107 (B2_IO)
- net BUSACK#: now also U6.13 (B10); no longer U8.20 (B3)
- net BUSREQ#: now also U6.14 (B9); no longer U8.21 (B2)
- net CART_CE#: now also U14.20 (B2); no longer U14.4 (A2)
- net D0: now also U4.20 (B3); no longer U4.16 (B7)
- net D1: now also U4.19 (B4); no longer U4.15 (B8)
- net D2: now also U4.18 (B5); no longer U4.14 (B9)
- net D3: now also U4.17 (B6); no longer U4.13 (B10)
- net D4: now also U4.16 (B7); no longer U6.22 (B1)
- net D5: now also U4.15 (B8); no longer U6.21 (B2)
- net D6: now also U4.14 (B9); no longer U6.20 (B3)
- net D7: now also U4.13 (B10); no longer U6.19 (B4)
- net DE_OE#: now also U1.83 (B3_IO); no longer U1.63 (B4_IO)
- net FPGA_A0: now also U1.131 (B0_IO), U2.8 (A7); no longer U1.141 (B0_IO), U2.2 (A1)
- net FPGA_A1: now also U1.130 (B0_IO), U2.9 (A8); no longer U1.140 (B0_IO), U2.3 (A2)
- net FPGA_A10: now also U1.118 (B1_IO), U8.8 (A7); no longer U1.116 (B1_IO), U4.2 (A1)
- net FPGA_A11: now also U1.116 (B1_IO), U8.9 (A8); no longer U1.113 (B1_IO), U4.3 (A2)
- net FPGA_A12: now also U1.113 (B1_IO), U8.10 (A9); no longer U1.112 (B1_IO), U4.4 (A3)
- net FPGA_A13: now also U1.112 (B1_IO), U8.11 (A10); no longer U1.119 (B1_IO), U4.5 (A4)
- net FPGA_A14: now also U1.108 (B2_IO), U4.2 (A1); no longer U1.118 (B1_IO), U4.6 (A5)
- net FPGA_A15: now also U1.107 (B2_IO), U4.3 (A2); no longer U1.123 (B1_IO_VREF), U4.7 (A6)
- net FPGA_A2: now also U1.129 (B0_IO_VREF), U2.10 (A9); no longer U1.137 (B0_IO), U2.4 (A3)
- net FPGA_A3: now also U1.128 (B0_IO_GCLK7), U2.11 (A10); no longer U1.135 (B0_IO), U2.5 (A4)
- net FPGA_A4: now also U1.127 (B0_IO_GCLK6), U8.2 (A1); no longer U1.132 (B0_IO), U2.6 (A5)
- net FPGA_A5: now also U1.125 (B1_IO_GCLK5), U8.3 (A2); no longer U1.131 (B0_IO), U2.7 (A6)
- net FPGA_A6: now also U1.124 (B1_IO_GCLK4), U8.4 (A3); no longer U1.130 (B0_IO), U2.8 (A7)
- net FPGA_A7: now also U1.123 (B1_IO_VREF), U8.5 (A4); no longer U1.129 (B0_IO_VREF), U2.9 (A8)
- net FPGA_A8: now also U1.122 (B1_IO), U8.6 (A5); no longer U1.128 (B0_IO_GCLK7), U2.10 (A9)
- net FPGA_A9: now also U1.119 (B1_IO), U8.7 (A6); no longer U1.127 (B0_IO_GCLK6), U2.11 (A10)
- net FPGA_BUSACK#: now also U1.84 (B3_IO_VREF), U6.11 (A10); no longer U1.80 (B3_IO), U8.4 (A3)
- net FPGA_BUSREQ#: now also U1.85 (B3_IO), U6.10 (A9); no longer U1.77 (B3_IO), U8.3 (A2)
- net FPGA_CART_CE#: now also U1.69 (B4_IO), U14.4 (A2); no longer U1.85 (B3_IO), U14.20 (B2)
- net FPGA_D0: now also U4.4 (A3); no longer U4.8 (A7)
- net FPGA_D1: now also U4.5 (A4); no longer U4.9 (A8)
- net FPGA_D2: now also U4.6 (A5); no longer U4.10 (A9)
- net FPGA_D3: now also U4.7 (A6); no longer U4.11 (A10)
- net FPGA_D4: now also U4.8 (A7); no longer U6.2 (A1)
- net FPGA_D5: now also U4.9 (A8); no longer U6.3 (A2)
- net FPGA_D6: now also U4.10 (A9); no longer U6.4 (A3)
- net FPGA_D7: now also U4.11 (A10); no longer U6.5 (A4)
- net FPGA_DE0: now also U1.82 (B3_IO); no longer U1.84 (B3_IO_VREF)
- net FPGA_DE1: now also U1.80 (B3_IO); no longer U1.87 (B3_IO)
- net FPGA_DE2: now also U1.79 (B3_IO); no longer U1.86 (B3_IO)
- net FPGA_DE3: now also U1.78 (B3_IO); no longer U1.90 (B3_IO_VREF)
- net FPGA_DE4: now also U1.77 (B3_IO); no longer U1.89 (B3_IO)
- net FPGA_DE5: now also U1.76 (B3_IO); no longer U1.70 (B4_IO_VREF)
- net FPGA_DE6: now also U1.74 (B3_IO); no longer U1.69 (B4_IO)
- net FPGA_DE7: now also U1.73 (B3_IO); no longer U1.68 (B4_IO)
- net FPGA_INT#: now also U1.87 (B3_IO), U6.8 (A7); no longer U1.73 (B3_IO), U8.2 (A1)
- net FPGA_IORQ#: now also U6.4 (A3); no longer U6.8 (A7)
- net FPGA_M1#: now also U6.2 (A1); no longer U6.6 (A5)
- net FPGA_MREQ#: now also U6.3 (A2); no longer U6.7 (A6)
- net FPGA_PHI: now also U1.70 (B4_IO_VREF), U14.3 (A1); no longer U1.82 (B3_IO), U14.21 (B1)
- net FPGA_RD#: now also U6.5 (A4); no longer U6.9 (A8)
- net FPGA_RESET#: now also U1.86 (B3_IO), U6.9 (A8); no longer U1.78 (B3_IO), U8.5 (A4)
- net FPGA_WAIT#: now also U1.89 (B3_IO), U6.7 (A6); no longer U1.74 (B3_IO), U6.11 (A10)
- net FPGA_WR#: now also U1.90 (B3_IO_VREF), U6.6 (A5); no longer U1.76 (B3_IO), U6.10 (A9)
- net GND: now also D1.2 (A), D2.2 (A), J14.10 (Pin_10), J16.10 (Pin_10); no longer U14.2 (DIR)
- net INT#: now also U6.16 (B7); no longer U8.22 (B1)
- net IORQ#: now also U6.20 (B3); no longer U6.16 (B7)
- net M1#: now also U6.22 (B1); no longer U6.18 (B5)
- net MREQ#: now also U6.21 (B2); no longer U6.17 (B6)
- net PHI: now also U14.21 (B1); no longer U14.3 (A1)
- net RAM_CE#: now also U1.68 (B4_IO); no longer U1.79 (B3_IO)
- net RD#: now also U6.19 (B4); no longer U6.15 (B8)
- net RESET#: now also U6.15 (B8); no longer U8.19 (B4)
- net ROM_CE#: now also U1.63 (B4_IO); no longer U1.83 (B3_IO)
- net USBCLK: now also U1.53 (B5_IO_GCLK3); no longer U1.52 (B5_IO_GCLK2)
- net USB_DM1: now also U1.18 (B7_IO_VREF); no longer U1.15 (B7_IO)
- net USB_DM2: now also U1.21 (B6_IO); no longer U1.18 (B7_IO_VREF)
- net USB_DP1: now also U1.20 (B6_IO_VREF); no longer U1.14 (B7_IO)
- net USB_DP2: now also U1.23 (B6_IO); no longer U1.17 (B7_IO)
- net VBUS: now also J13.1 (VBUS); no longer J9.1 (VBUS)
- net VGA_B0: now also U1.4 (B7_IO_VREF); no longer U1.8 (B7_IO)
- net VGA_B1: now also U1.5 (B7_IO); no longer U1.7 (B7_IO)
- net VGA_B2: now also U1.6 (B7_IO); no longer U1.11 (B7_IO)
- net VGA_B3: now also U1.7 (B7_IO); no longer U1.10 (B7_IO)
- net VGA_G0: now also U1.8 (B7_IO); no longer U1.2 (B7_IO)
- net VGA_G1: now also U1.10 (B7_IO); no longer U1.1 (B7_IO)
- net VGA_G2: now also U1.11 (B7_IO); no longer U1.6 (B7_IO)
- net VGA_G3: now also U1.12 (B7_IO); no longer U1.5 (B7_IO)
- net VGA_HSYNC: now also U1.1 (B7_IO); no longer U1.13 (B7_IO)
- net VGA_R0: now also U1.13 (B7_IO); no longer U1.23 (B6_IO)
- net VGA_R1: now also U1.14 (B7_IO); no longer U1.21 (B6_IO)
- net VGA_R2: now also U1.15 (B7_IO); no longer U1.20 (B6_IO_VREF)
- net VGA_R3: now also U1.17 (B7_IO); no longer U1.4 (B7_IO_VREF)
- net VGA_VSYNC: now also U1.2 (B7_IO); no longer U1.12 (B7_IO)
- net WAIT#: now also U6.17 (B6); no longer U6.13 (B10)
- net WR#: now also U6.18 (B5); no longer U6.14 (B9)
- net at Q2.1 (B), R30.2, R31.1: now also D2.1 (K)
- net at R86.2, R94.1: now also U12.4 (C); no longer U12.5 (D)
- net at R87.2, R95.1: now also U12.12 (G); no longer U12.10 (E)
- net FPGA_EXP2: now reaches U1.50 (B5_IO)
- net FPGA_EXP2: now also J14.4 (Pin_4)
- net at R61.2, R69.1: now also U9.14 (H); no longer U9.12 (G)
- net ESP_EXP7: now reaches U5.30 (IO37)
- net ESP_EXP7: now also J16.9 (Pin_9)
- net ESP_EXP6: now reaches U5.31 (IO38)
- net ESP_EXP6: now also J16.8 (Pin_8)
- net ESP_EXP5: now reaches U5.32 (IO39)
- net ESP_EXP5: now also J16.7 (Pin_7)
- net ESP_EXP4: now reaches U5.33 (IO40)
- net ESP_EXP4: now also J16.6 (Pin_6)
- net ESP_EXP3: now reaches U5.34 (IO41)
- net ESP_EXP3: now also J16.5 (Pin_5)
- net ESP_EXP2: now reaches U5.35 (IO42)
- net ESP_EXP2: now also J16.4 (Pin_4)
- net ESP_EXP1: now reaches U5.38 (IO2)
- net ESP_EXP1: now also J16.3 (Pin_3)
- net ESP_EXP0: now reaches U5.39 (IO1)
- net ESP_EXP0: now also J16.2 (Pin_2)
- net at R56.2, R64.1: now also U9.5 (D); no longer U9.3 (B)
- net at R57.2, R65.1: now also U9.11 (F); no longer U9.4 (C)
- net at R60.2, R68.1: now also U9.3 (B); no longer U9.11 (F)
- net at R85.2, R93.1: now also U12.11 (F); no longer U12.4 (C)
- net at R55.2, R63.1: now also U9.10 (E); no longer U9.2 (A)
- net at R62.2, R70.1: now also U9.2 (A); no longer U9.14 (H)
- net at R59.2, R67.1: now also U9.12 (G); no longer U9.10 (E)
- net at R88.2, R96.1: now also U12.3 (B); no longer U12.11 (F)
- net at U14.10 (A8): now also U14.7 (A5), U14.8 (A6), U14.9 (A7)
- net at R90.2, R98.1: now also U12.2 (A); no longer U12.14 (H)
- net at C33.2, Q1.1 (B), R25.1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: now also D1.1 (K)
- net at R83.2, R91.1: now also U12.10 (E); no longer U12.2 (A)
- net at R84.2, R92.1: now also U12.5 (D); no longer U12.3 (B)
- net at R58.2, R66.1: now also U9.4 (C); no longer U9.5 (D)
- net at R89.2, R97.1: now also U12.14 (H); no longer U12.12 (G)
- net CVID0 renamed FPGA_EXP1
- net FPGA_EXP1: now also J14.3 (Pin_3)
- net CVID1 renamed FPGA_EXP4
- net FPGA_EXP4: now also J14.6 (Pin_6)
- net CVID2 renamed FPGA_EXP3
- net FPGA_EXP3: now also J14.5 (Pin_5)
- net CVID3 renamed FPGA_EXP7
- net FPGA_EXP7: now also J14.9 (Pin_9)
- net CVID4 renamed FPGA_EXP6
- net FPGA_EXP6: now also J14.8 (Pin_8)
- net CVID5 renamed FPGA_EXP5
- net FPGA_EXP5: now also J14.7 (Pin_7)
- new net FPGA_EXP0: J14.2 (Pin_2), U1.52 (B5_IO_GCLK2)
- no-connect marks 14 -> 22
Other:
- note added: "Activity LED"
- note added: "Spare ESP32 pins"
- note added: "Spare FPGA pins"
- note removed: "Composite video output"
- note removed: "LEDs"
- moved on the sheet: C42, C43, C47, C50, C51, C53, C54, C58, D4, J11, R47, R48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

Commit message: Working on layout.
Connections:
- net SND is gone; now on net CASSETTE_OUT: J15.2 (Pin_2)
- net AUDIO_L: now also U1.20 (B6_IO_VREF); no longer U1.25 (B6_IO)
- net AUDIO_R: now also U1.18 (B7_IO_VREF); no longer U1.24 (B6_IO_VREF)
- net CASSETTE_IN: now also U1.23 (B6_IO); no longer U1.32 (B6_IO)
- net CASSETTE_OUT: now also U1.21 (B6_IO); no longer U1.31 (B6_IO)
- net ESP_CTS: now also U5.24 (IO33); no longer U5.20 (IO12)
- net ESP_NOTIFY: now also U1.31 (B6_IO), U5.20 (IO12); no longer U1.36 (B6_IO), U5.10 (IO17)
- net ESP_RTS: now also U5.22 (IO14); no longer U5.18 (IO10)
- net ESP_RX: now also U5.23 (IO21); no longer U5.19 (IO11)
- net ESP_TX: now also U5.21 (IO13); no longer U5.17 (IO9)
- net FPGA_DONE: now also U5.12 (IO8); no longer U5.9 (IO16)
- net FPGA_PROG#: now also U5.25 (IO34); no longer U5.8 (IO15)
- net PRINTER_IN: now also U1.24 (B6_IO_VREF); no longer U1.33 (B6_IO)
- net PRINTER_OUT: now also U1.25 (B6_IO); no longer U1.35 (B6_IO)
- net SD_ACTIVITY: now also U5.4 (IO4); no longer U5.29 (IO36)
- net SD_CD#: now also U5.6 (IO6); no longer U5.28 (IO35)
- net SD_MISO: now also U5.7 (IO7); no longer U5.21 (IO13)
- net SD_MOSI: now also U5.9 (IO16); no longer U5.22 (IO14)
- net SD_SCK: now also U5.8 (IO15); no longer U5.23 (IO21)
- net SD_SSEL#: now also U5.10 (IO17); no longer U5.24 (IO33)
- net SD_WP#: now also U5.5 (IO5); no longer U5.25 (IO34)
- net SPI_CS#: now also U5.19 (IO11); no longer U5.4 (IO4)
- net SPI_MISO: now also U5.15 (IO3); no longer U5.7 (IO7)
- net SPI_MOSI: now also U5.17 (IO9); no longer U5.6 (IO6)
- net SPI_SCLK: now also U5.18 (IO10); no longer U5.5 (IO5)
- net USB_DM1: now also U1.35 (B6_IO); no longer U1.18 (B7_IO_VREF)
- net USB_DM2: now also U1.32 (B6_IO); no longer U1.21 (B6_IO)
- net USB_DP1: now also U1.36 (B6_IO); no longer U1.20 (B6_IO_VREF)
- net USB_DP2: now also U1.33 (B6_IO); no longer U1.23 (B6_IO)

Commit message: Working on PCB layout.
Connections:
- net FPGA_CART_CE#: now also U1.70 (B4_IO_VREF); no longer U1.69 (B4_IO)
- net FPGA_PHI: now also U1.69 (B4_IO); no longer U1.70 (B4_IO_VREF)
- net GND: now also U14.10 (A8), U14.5 (A3), U14.6 (A4), U14.7 (A5), U14.8 (A6), U14.9 (A7)
- no-connect marks 22 -> 20
Changed lines of the file:
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@@
   (junction (at 422.91 25.4) (diameter 0) (color 0 0 0 0)
   )
+  (junction (at 370.84 252.73) (diameter 0) (color 0 0 0 0)
+  )
   (junction (at 121.92 107.95) (diameter 0) (color 0 0 0 0)
   )
@@
   (junction (at 44.45 257.81) (diameter 0) (color 0 0 0 0)
   )
+  (junction (at 370.84 250.19) (diameter 0) (color 0 0 0 0)
+  )
   (junction (at 486.41 63.5) (diameter 0) (color 0 0 0 0)
   )
@@
   (junction (at 44.45 267.97) (diameter 0) (color 0 0 0 0)
   )
+  (junction (at 370.84 247.65) (diameter 0) (color 0 0 0 0)
+  )
   (junction (at 44.45 228.6) (diameter 0) (color 0 0 0 0)
   )
@@
   (no_connect (at 435.61 27.94))
   (no_connect (at 434.34 40.64))
-  (no_connect (at 372.11 250.19))
-  (no_connect (at 372.11 247.65))
   (no_connect (at 207.01 62.23))
   (no_connect (at 309.88 152.4))
@@
     (stroke (width 0) (type default) (color 0 0 0 0))
   )
+  (wire (pts (xy 370.84 250.19) (xy 370.84 252.73))
+    (stroke (width 0) (type default) (color 0 0 0 0))
+  )
   (wire (pts (xy 130.81 289.56) (xy 132.08 289.56))
     (stroke (width 0) (type default) (color 0 0 0 0))
@@
     (stroke (width 0) (type default) (color 0 0 0 0))
   )
+  (wire (pts (xy 370.84 247.65) (xy 370.84 250.19))
+    (stroke (width 0) (type default) (color 0 0 0 0))
+  )
   (polyline (pts (xy 412.75 223.52) (xy 412.75 279.4))
     (stroke (width 0) (type solid) (color 0 0 0 0))
@@
     (stroke (width 0) (type default) (color 0 0 0 0))
   )
+  (wire (pts (xy 370.84 247.65) (xy 367.03 247.65))
+    (stroke (width 0) (type default) (color 0 0 0 0))
+  )
   (wire (pts (xy 139.7 120.65) (xy 140.97 120.65))
     (stroke (width 0) (type default) (color 0 0 0 0))
@@
     (stroke (width 0) (type default) (color 0 0 0 0))
   )
+  (wire (pts (xy 372.11 247.65) (xy 370.84 247.65))
+    (stroke (width 0) (type default) (color 0 0 0 0))
+  )
   (wire (pts (xy 115.57 189.23) (xy 115.57 186.69))
     (stroke (width 0) (type default) (color 0 0 0 0))
@@
     (stroke (width 0) (type default) (color 0 0 0 0))
   )
+  (wire (pts (xy 367.03 247.65) (xy 367.03 248.92))
+    (stroke (width 0) (type default) (color 0 0 0 0))
+  )
   (wire (pts (xy 186.69 120.65) (xy 187.96 120.65))
     (stroke (width 0) (type default) (color 0 0 0 0))
@@
     (stroke (width 0) (type default) (color 0 0 0 0))
   )
+  (wire (pts (xy 370.84 250.19) (xy 372.11 250.19))
+    (stroke (width 0) (type default) (color 0 0 0 0))
+  )
   (wire (pts (xy 123.19 123.19) (xy 119.38 123.19))
     (stroke (width 0) (type default) (color 0 0 0 0))
@@
     )
   )
-  (global_label "FPGA_PHI" (shape output) (at 81.28 157.48 0) (fields_autoplaced)
+  (global_label "FPGA_PHI" (shape output) (at 81.28 160.02 0) (fields_autoplaced)
     (effects (font (size 1.27 1.27)) (justify left))
-    (property "Intersheet References" "${INTERSHEET_REFS}" (id 0) (at 92.5831 157.4006 0)
+    (property "Intersheet References" "${INTERSHEET_REFS}" (id 0) (at 92.5831 159.9406 0)
       (effects (font (size 1.27 1.27)) (justify left) hide)
     )
@@
     )
   )
-  (global_label "FPGA_CART_CE#" (shape output) (at 81.28 160.02 0) (fields_autoplaced)
+  (global_label "FPGA_CART_CE#" (shape output) (at 81.28 157.48 0) (fields_autoplaced)
     (effects (font (size 1.27 1.27)) (justify left))
-    (property "Intersheet References" "${INTERSHEET_REFS}" (id 0) (at 98.6307 159.9406 0)
+    (property "Intersheet References" "${INTERSHEET_REFS}" (id 0) (at 98.6307 157.4006 0)
       (effects (font (size 1.27 1.27)) (justify left) hide)
     )
@@
     (pin "2")
   )
+  (symbol (lib_id "power:GND") (at 367.03 248.92 0) (mirror y) (unit 1)
+    (in_bom yes) (on_board yes)
+    (property "Reference" "#PWR?" (id 0) (at 367.03 255.27 0)
+      (effects (font (size 1.27 1.27)) hide)
+    )
+    (property "Value" "GND" (id 1) (at 367.03 252.73 0))
+    (property "Footprint" "" (id 2) (at 367.03 248.92 0)
+      (effects (font (size 1.27 1.27)) hide)
+    )
+    (property "Datasheet" "" (id 3) (at 367.03 248.92 0)
+      (effects (font (size 1.27 1.27)) hide)
+    )
+    (pin "1")
+  )
   (symbol (lib_id "Device:R") (at 127 107.95 90) (unit 1)
     (in_bom yes) (on_board yes)
@@
       (reference "#PWR0178") (unit 1) (value "GND") (footprint "")
     )
+    (path "/d570a76b-ebb0-4d7d-9564-6c977401c409"
+      (reference "#PWR?") (unit 1) (value "GND") (footprint "")
+    )
     (path "/52d4c05f-c0de-4113-8daf-5e4446b453ca"
