File: pcb/rev2/aquarius-plus.kicad_pcb (KiCad board)
At the start: 2 copper layers, 167 x 115 mm, 173 parts, among them J1 Power in, J10 FPGA spare, J11 Hand controller 2, J12 Hand controller 1, J13 ESP32 spare, J2 ESP USB Host, J3 Audio out, J4 VGA, J5 Cassette out, J6 Cassette in, J7 Expansion port, J8 Printer, J9 TF-03A, Q1 BC847C, Q2 BC847C, Q3 2N7002, SW1 SW_DPDT_x2, U1 SN74AHCT1G125DBVR, U10 ESP32-S3-WROOM-1-N4R2, U11 LDL1117S33R, U12 SN74CB3T3245PWR, U13 IS61C5128AS-25QLI, U2 SN74AHCT1G125DBVR, U3 LD1117S12, U4 SN74CB3T3245PWR, U5 MAX3221ECPWR, U6 XC6SLX9-2TQG144C, U7 Z84C0010AEG, U8 SN74CB3T3245PWR, U9 SN74CB3T3245PWR, X1 SX3M14.31818M20F30TNN

Commit message: Update
Parts:
- J3, J5, J6, J8: footprint Connector_Audio:Jack_3.5mm_CUI_SJ-3523-SMT_Horizontal -> aquarius-plus:C2884998
- moved J3 1.00 mm to (125.0, 40.0)
- moved J5 1.00 mm to (70.0, 49.0)
- moved J6 1.00 mm to (70.0, 64.0)
- moved J8 1.00 mm to (70.0, 79.0)
Routing:
- net Net-(J5-PadR): track 21.2 -> 24.6 mm
- net Net-(U5-DOUT): track 22.2 -> 25.1 mm
- net Net-(C1-Pad2): track 6.24 -> 8.88 mm
- net VBUS: track 126.7 -> 128.9 mm
- net Net-(U5-RIN): track 26.2 -> 27.9 mm
- net Net-(J6-PadT): track 9.18 -> 10.6 mm
- net GND: track 116.2 -> 115.7 mm
- net Net-(J6-PadR): track 12.5 -> 13.0 mm

Commit message: PCB Updates
Routing:
- net VBUS: track 128.9 -> 135.5 mm
- net +5V: track 484.1 -> 480.8 mm
Changed lines of the file:
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@@
     (fp_rect (start -2.5 -7.75) (end 2.5 -5)
       (stroke (width 0.12) (type default)) (fill none) (layer "F.SilkS"))
-    (pad "" np_thru_hole circle (at 0 -2.9 90) (size 1.6 1.6) (drill 0.8) (layers "F&B.Cu" "*.Mask"))
-    (pad "" np_thru_hole circle (at 0 4.1 90) (size 1.6 1.6) (drill 0.8) (layers "F&B.Cu" "*.Mask"))
+    (pad "" np_thru_hole circle (at 0 -2.9 90) (size 1.2 1.2) (drill 0.8) (layers "F&B.Cu" "*.Mask"))
+    (pad "" np_thru_hole circle (at 0 3.1 90) (size 1.2 1.2) (drill 0.8) (layers "F&B.Cu" "*.Mask"))
     (pad "R" smd roundrect (at 4 -0.98 90) (size 3 2) (layers "F.Cu" "F.Paste" "F.Mask") (roundrect_rratio 0.25)
       (net 211 "Net-(J6-PadR)") (pintype "passive") (thermal_bridge_angle 45))
@@
     (fp_rect (start -2.5 -7.75) (end 2.5 -5)
       (stroke (width 0.12) (type default)) (fill none) (layer "F.SilkS"))
-    (pad "" np_thru_hole circle locked (at 0 -2.9 90) (size 1.6 1.6) (drill 0.8) (layers "F&B.Cu" "*.Mask"))
-    (pad "" np_thru_hole circle locked (at 0 4.1 90) (size 1.6 1.6) (drill 0.8) (layers "F&B.Cu" "*.Mask"))
+    (pad "" np_thru_hole circle locked (at 0 -2.9 90) (size 1.2 1.2) (drill 0.8) (layers "F&B.Cu" "*.Mask"))
+    (pad "" np_thru_hole circle locked (at 0 3.1 90) (size 1.2 1.2) (drill 0.8) (layers "F&B.Cu" "*.Mask"))
     (pad "R" smd roundrect locked (at 4 -0.98 90) (size 3 2) (layers "F.Cu" "F.Paste" "F.Mask") (roundrect_rratio 0.25)
       (net 214 "Net-(U5-RIN)") (pintype "passive") (thermal_bridge_angle 45))
@@
     (fp_rect (start -2.5 -7.75) (end 2.5 -5)
       (stroke (width 0.12) (type default)) (fill none) (layer "F.SilkS"))
-    (pad "" np_thru_hole circle (at 0 -2.9) (size 1.6 1.6) (drill 0.8) (layers "F&B.Cu" "*.Mask"))
-    (pad "" np_thru_hole circle (at 0 4.1) (size 1.6 1.6) (drill 0.8) (layers "F&B.Cu" "*.Mask"))
+    (pad "" np_thru_hole circle (at 0 -2.9) (size 1.2 1.2) (drill 0.8) (layers "F&B.Cu" "*.Mask"))
+    (pad "" np_thru_hole circle (at 0 3.1) (size 1.2 1.2) (drill 0.8) (layers "F&B.Cu" "*.Mask"))
     (pad "R" smd roundrect (at 4 -0.98) (size 3 2) (layers "F.Cu" "F.Paste" "F.Mask") (roundrect_rratio 0.25)
       (net 185 "Net-(C3-Pad2)") (pintype "passive") (thermal_bridge_angle 45))
@@
     (fp_rect (start -2.5 -7.75) (end 2.5 -5)
       (stroke (width 0.12) (type default)) (fill none) (layer "F.SilkS"))
-    (pad "" np_thru_hole circle (at 0 -2.9 90) (size 1.6 1.6) (drill 0.8) (layers "F&B.Cu" "*.Mask"))
-    (pad "" np_thru_hole circle (at 0 4.1 90) (size 1.6 1.6) (drill 0.8) (layers "F&B.Cu" "*.Mask"))
+    (pad "" np_thru_hole circle (at 0 -2.9 90) (size 1.2 1.2) (drill 0.8) (layers "F&B.Cu" "*.Mask"))
+    (pad "" np_thru_hole circle (at 0 3.1 90) (size 1.2 1.2) (drill 0.8) (layers "F&B.Cu" "*.Mask"))
     (pad "R" smd roundrect (at 4 -0.98 90) (size 3 2) (layers "F.Cu" "F.Paste" "F.Mask") (roundrect_rratio 0.25)
       (net 210 "Net-(J5-PadR)") (pintype "passive") (thermal_bridge_angle 45))
@@
   (via (at 181.720763 112.226) (size 0.6) (drill 0.3) (layers "F.Cu" "B.Cu") (net 2))
   (via (at 144.644203 88.441725) (size 0.6) (drill 0.3) (layers "F.Cu" "B.Cu") (net 2))
-  (via (at 134.35153 41.382264) (size 0.6) (drill 0.3) (layers "F.Cu" "B.Cu") (free) (net 2))
+  (via (at 137.16 41.382264) (size 0.6) (drill 0.3) (layers "F.Cu" "B.Cu") (free) (net 2))
   (via (at 113.331833 74.55) (size 0.6) (drill 0.3) (layers "F.Cu" "B.Cu") (net 2))
   (via (at 190.5 129.54) (size 0.6) (drill 0.3) (layers "F.Cu" "B.Cu") (free) (net 2))
@@
   (via (at 141.15 117.65) (size 0.6) (drill 0.3) (layers "F.Cu" "B.Cu") (free) (net 2))
   (via (at 117.298483 41.825531) (size 0.6) (drill 0.3) (layers "F.Cu" "B.Cu") (free) (net 2))
-  (via (at 114.657222 53.319907) (size 0.6) (drill 0.3) (layers "F.Cu" "B.Cu") (free) (net 2))
+  (via (at 113.03 50.8) (size 0.6) (drill 0.3) (layers "F.Cu" "B.Cu") (free) (net 2))
   (via (at 150.762568 91.015104) (size 0.6) (drill 0.3) (layers "F.Cu" "B.Cu") (net 2))
   (via (at 96.649603 121.75062) (size 0.6) (drill 0.3) (layers "F.Cu" "B.Cu") (net 2))
@@
   (via (at 166.85 68.15) (size 0.6) (drill 0.3) (layers "F.Cu" "B.Cu") (net 5))
   (segment (start 117.55 117.5) (end 116 115.95) (width 1) (layer "B.Cu") (net 5))
-  (segment (start 120.45 41.55) (end 129.65 41.55) (width 1) (layer "B.Cu") (net 5))
-  (segment (start 111.9 55.88) (end 111.9 50.1) (width 1) (layer "B.Cu") (net 5))
   (segment (start 179.3 118.3) (end 178.45 117.45) (width 0.5) (layer "B.Cu") (net 5))
-  (segment (start 198.2 48.7) (end 204.59 48.7) (width 1) (layer "B.Cu") (net 5))
   (segment (start 201.55 76.05) (end 201.55 64.2381) (width 0.5) (layer "B.Cu") (net 5))
   (segment (start 178.45 117.45) (end 178.45 112.3) (width 0.5) (layer "B.Cu") (net 5))
-  (segment (start 132.85 38.35) (end 187.85 38.35) (width 1) (layer "B.Cu") (net 5))
+  (segment (start 111.9 55.74) (end 118.11 49.53) (width 1) (layer "B.Cu") (net 5))
+  (segment (start 204.59 48.7) (end 208.9575 44.3325) (width 1) (layer "B.Cu") (net 5))
+  (segment (start 111.9 55.88) (end 111.9 55.74) (width 1) (layer "B.Cu") (net 5))
+  (segment (start 127 49.53) (end 138.18 38.35) (width 1) (layer "B.Cu") (net 5))
   (segment (start 166.85 68.15) (end 166.85 64.2381) (width 0.5) (layer "B.Cu") (net 5))
   (segment (start 128.1 117.5) (end 117.55 117.5) (width 1) (layer "B.Cu") (net 5))
-  (segment (start 111.9 50.1) (end 120.45 41.55) (width 1) (layer "B.Cu") (net 5))
-  (segment (start 129.65 41.55) (end 132.85 38.35) (width 1) (layer "B.Cu") (net 5))
-  (segment (start 204.59 48.7) (end 208.9575 44.3325) (width 1) (layer "B.Cu") (net 5))
+  (segment (start 138.18 38.35) (end 187.85 38.35) (width 1) (layer "B.Cu") (net 5))
   (segment (start 187.85 38.35) (end 198.2 48.7) (width 1) (layer "B.Cu") (net 5))
+  (segment (start 118.11 49.53) (end 127 49.53) (width 1) (layer "B.Cu") (net 5))
+  (segment (start 198.2 48.7) (end 204.59 48.7) (width 1) (layer "B.Cu") (net 5))
   (segment (start 89.375 70.65) (end 89.375 72.1) (width 0.3) (layer "F.Cu") (net 6))
   (segment (start 89.8875 70.1375) (end 89.375 70.65) (width 0.3) (layer "F.Cu") (net 6))
@@
   (via (at 84.8 38.05) (size 0.6) (drill 0.3) (layers "F.Cu" "B.Cu") (net 87))
   (segment (start 199.575 36.45) (end 204.9575 41.8325) (width 1) (layer "B.Cu") (net 87))
-  (segment (start 121.415259 36.45) (end 124.058237 39.092978) (width 1) (layer "B.Cu") (net 87))
-  (segment (start 88.3 38.05) (end 89.9 36.45) (width 1) (layer "B.Cu") (net 87))
-  (segment (start 124.058237 39.092978) (end 125.892298 39.092978) (width 1) (layer "B.Cu") (net 87))
+  (segment (start 119.45 47.06) (end 126.502944 47.06) (width 1) (layer "B.Cu") (net 87))
   (segment (start 84.8 38.05) (end 88.3 38.05) (width 1) (layer "B.Cu") (net 87))
-  (segment (start 89.9 36.45) (end 121.415259 36.45) (width 1) (layer "B.Cu") (net 87))
+  (segment (start 88.3 38.05) (end 89.9 36.45) (width 1) (layer "B.Cu") (net 87))
+  (segment (start 126.502944 47.06) (end 137.112944 36.45) (width 1) (layer "B.Cu") (net 87))
+  (segment (start 89.9 36.45) (end 108.84 36.45) (width 1) (layer "B.Cu") (net 87))
+  (segment (start 108.84 36.45) (end 119.45 47.06) (width 1) (layer "B.Cu") (net 87))
   (segment (start 204.9575 41.8325) (end 204.9575 44.3325) (width 1) (layer "B.Cu") (net 87))
-  (segment (start 128.535276 36.45) (end 199.575 36.45) (width 1) (layer "B.Cu") (net 87))
-  (segment (start 125.892298 39.092978) (end 128.535276 36.45) (width 1) (layer "B.Cu") (net 87))
+  (segment (start 137.112944 36.45) (end 199.575 36.45) (width 1) (layer "B.Cu") (net 87))
   (segment (start 123.405249 87.9625) (end 123.177099 87.73435) (width 0.2) (layer "F.Cu") (net 88))
   (segment (start 110.462984 87.101996) (end 112.312984 87.101996) (width 0.2) (layer "F.Cu") (net 88))
